Commit message: First stable release.

File: urdf/kuka_kr16.urdf (robot description, URDF)
Before this commit: robot kuka_kr16, 3 links, 2 joints
Links:
- removed link base
- removed link base_link
- removed link link_1
- added link ${prefix}tool0
Joints:
- removed joint base_link-base
- removed joint joint_a1
